File: ICM-45686.kicad_sch (KiCad schematic)
At the start: 0 parts

Commit message: 回路図とPCBの作成
Parts:
- added C1: 1uF X7R, Capacitor_SMD:C_0402_1005Metric, symbol Device:C_Small
- added C2, C3: 100nF X7R, Capacitor_SMD:C_0402_1005Metric, symbol Device:C_Small
- added J1, J2: Conn_01x04_Pin, Connector_PinHeader_2.54mm:PinHeader_1x04_P2.54mm_Vertical, symbol Connector:Conn_01x04_Pin
- added U1: ICM-45686, ICM_45686:IC_ICM-45686, symbol ICM-45686:ICM-45686
Connections:
- new net +3.3V: C1.1, C2.1, C3.1, J1.1 (Pin_1), U1.5 (VDDIO), U1.8 (VDD)
- new net CS: J2.4 (Pin_4), U1.12 (AP_CS)
- new net FSYNC: J2.2 (Pin_2), U1.9 (INT2/FSYNC/CLKIN)
- new net GND: C1.2, C2.2, C3.2, J1.2 (Pin_2), U1.6 (GND)
- new net INT: J2.1 (Pin_1), U1.4 (INT1/INT)
- new net MISO: J1.4 (Pin_4), U1.1 (AP_SDO/AP_AD0)
- new net MOSI: J2.3 (Pin_3), U1.14 (AP_SDA/AP_SDIO/AP_SDI)
- new net SCLK: J1.3 (Pin_3), U1.13 (AP_SCL/AP_SCLK)
- no-connect marks 0 -> 5
Other:
- company: (none) -> Koki
- title: (none) -> ICM-45686 Module
